Commit message: RVIZ commit 3
- Finished URDF file
- Updated to do list, moving to gazebo launch file

File: trashbot.urdf (robot description, URDF)
Before this commit: robot trashbot, 4 links, 3 joints
Links:
- added link base_scan, mass 0; collision cylinder length=0.0315 radius=0.055; visual mesh filename=package://trashbot_description/meshes/lds.stl scale=0.001 0.001 0.001
- added link imu_link
Joints:
- added joint imu_joint: type fixed, parent base_link, child imu_link, origin xyz=0 0 0.205 rpy=0 0 0
- added joint scan_joint: type fixed, parent base_link, child base_scan, origin xyz=0 0 0.205 rpy=0 0 0
