Commit message: RVIZ commit 1
- Fixed trashbot launch file
- Fixing trashbot urdf
- Added turtlebot3_burger launch, urdf and meshes for testing RVIZ and Gazebo
- Updated to do list

File: trashbot_description/urdf/trashbot.urdf (robot description, URDF)
Before this commit: robot trashbot, 4 links, 3 joints
Links:
- removed link base_scan
- removed link imu_link
- added link wheel_left_link, mass 2; collision cylinder length=0.05 radius=0.1; visual cylinder length=0.05 radius=0.1
- link base_link: geometry collision box size=0.2 0.4 0.15; visual box size=0.2 0.4 0.2
Joints:
- removed joint imu_joint
- removed joint scan_joint
- added joint wheel_left_joint: type continuous, parent base_link, child wheel_left_link, origin xyz=0 0 0 rpy=0 0 0, axis 0 0 0
- joint base_joint: origin xyz=0.0 0.0 0.010 rpy=0 0 0 -> xyz=0 0 0 rpy=0 0 0

Commit message: Trashbot URDF commit 1 - Added base scan and imu links and joints

File: trashbot_description/urdf/trashbot.urdf (robot description, URDF)
Before this commit: robot trashbot, 3 links, 2 joints
Links:
- added link base_scan, mass 0; collision cylinder length=0.0315 radius=0.055; visual mesh filename=package://trashbot_description/meshes/lds.stl scale=0.001 0.001 0.001
- added link imu_link
- added link wheel_right_link, mass 2; collision cylinder length=0.05 radius=0.1; visual cylinder length=0.05 radius=0.1
- link base_link: geometry collision box size=0.2 0.4 0.15; visual box size=0.2 0.4 0.15
Joints:
- added joint imu_joint: type fixed, parent base_link, child imu_link, origin xyz=0 0 0.205 rpy=0 0 0
- added joint scan_joint: type fixed, parent base_link, child base_scan, origin xyz=0 0 0.205 rpy=0 0 0
- added joint wheel_right_joint: type continuous, parent base_link, child wheel_right_link, origin xyz=0 -0.225 0.1 rpy=0 0 0, axis 0 1 0
- joint wheel_left_joint: axis 0 0 0 -> 0 1 0; origin xyz=0 0 0 rpy=0 0 0 -> xyz=0 0.225 0.1 rpy=0 0 0
